Commit message: Migrate simulation to ROS 2 Jazzy / Gazebo Harmonic
Port the sim from Gazebo Fortress (Ignition) to Gazebo Harmonic (gz-sim 8),
the ROS 2 Jazzy pairing, and replace the robot to fix wheel-odometry slip.

- Rename all system plugins: ignition-gazebo-*-system -> gz-sim-*-system and
  ignition::gazebo::systems -> gz::sim::systems, across the URDF and 5 worlds
- Replace the 4-wheel skid-steer with a clean 2-wheel differential drive plus
  two frictionless ball casters (olive_bot.urdf.xacro) for low-slip /odom
- Launch: use GZ_SIM_RESOURCE_PATH, bridge /clock for use_sim_time, and add a
  headless (server-only) option
- Consolidate to canonical filenames: simulation.launch.py,
  simulation_manual.launch.py, olive_bot.urdf.xacro, fusion_test_world.sdf
- Remove Gazebo Classic legacy files and the old skid-steer URDF
- Rewrite READMEs and config docs for Jazzy/Harmonic

File: urdf/olive_bot.urdf.xacro (robot description, xacro)
@@ -1,91 +1,116 @@
 <?xml version="1.0"?>
+<!--
+  olive_bot - clean 2-wheel differential-drive + caster robot for Gazebo Harmonic (ROS 2 Jazzy).
+  Replaces the old 4-wheel skid-steer, whose wheels slipped on every turn (and occasionally
+  "slept"), producing poor /odom. A differential drive with two frictionless ball casters
+  matches the DiffDrive plugin's kinematics exactly -> clean, low-slip wheel odometry.
+  Sensor suite (16-beam 3D LiDAR, 100 Hz IMU, RGB camera) and all topic names are unchanged.
+  Frames (REP-105 friendly): odom -> base_footprint -> base_link -> {sensors}.
+  DiffDrive publishes odom->base_footprint; robot_state_publisher publishes base_footprint->base_link.
+-->
 <robot xmlns:xacro="http://www.ros.org/wiki/xacro" name="olive_bot">
-  <!-- Define properties for easy modification -->
-  <xacro:property name="chassis_length" value="0.5"/>
-  <xacro:property name="chassis_width" value="0.3"/>
-  <xacro:property name="chassis_height" value="0.15"/>
-  <xacro:property name="wheel_radius" value="0.05"/>
-  <xacro:property name="wheel_width" value="0.04"/>
-  <xacro:property name="wheel_offset_x" value="0.15"/>
-  <xacro:property name="wheel_offset_y" value="0.17"/>
-  <xacro:property name="wheel_offset_z" value="-0.05"/>
-  <!-- Base footprint (for navigation stack compatibility) -->
+  <!-- ============================ Properties ============================ -->
+  <xacro:property name="chassis_length"  value="0.40"/>
+  <xacro:property name="chassis_width"   value="0.30"/>
+  <xacro:property name="chassis_height"  value="0.12"/>
+  <xacro:property name="chassis_mass"    value="10.0"/>
+  <xacro:property name="wheel_radius"    value="0.06"/>
+  <xacro:property name="wheel_width"     value="0.04"/>
+  <xacro:property name="wheel_mass"      value="0.5"/>
+  <xacro:property name="wheel_offset_y"  value="0.16"/>   <!-- half of wheel_separation -->
+  <xacro:property name="caster_radius"   value="0.03"/>
+  <xacro:property name="caster_mass"     value="0.1"/>
+  <xacro:property name="caster_offset_x" value="0.15"/>
+  <!-- ============================ Base ============================ -->
+  <!-- base_footprint sits on the ground; base_link is raised to wheel-axle height -->
   <link name="base_footprint"/>
   <joint name="base_joint" type="fixed">
     <parent link="base_footprint"/>
     <child link="base_link"/>
-    <origin xyz="0.0 0.0 ${wheel_radius}" rpy="0 0 0"/>
-  </joint>
-  <!-- Base Link (Chassis) -->
+    <origin xyz="0 0 ${wheel_radius}" rpy="0 0 0"/>
+  </joint>
   <link name="base_link">
     <visual>
-      <origin xyz="0 0 0" rpy="0 0 0"/>
-      <geometry>
-        <box size="${chassis_length} ${chassis_width} ${chassis_height}"/>
-      </geometry>
-      <material name="blue">
-        <color rgba="0.0 0.0 1.0 1.0"/>
-      </material>
+      <origin xyz="0 0 ${chassis_height/2}" rpy="0 0 0"/>
+      <geometry><box size="${chassis_length} ${chassis_width} ${chassis_height}"/></geometry>
+      <material name="blue"><color rgba="0.0 0.0 1.0 1.0"/></material>
     </visual>
     <collision>
-      <origin xyz="0 0 0" rpy="0 0 0"/>
-      <geometry>
-        <box size="${chassis_length} ${chassis_width} ${chassis_height}"/>
-      </geometry>
+      <origin xyz="0 0 ${chassis_height/2}" rpy="0 0 0"/>
+      <geometry><box size="${chassis_length} ${chassis_width} ${chassis_height}"/></geometry>
     </collision>
     <inertial>
-      <mass value="15.0"/>
-      <origin xyz="0 0 0" rpy="0 0 0"/>
-      <inertia ixx="0.1125" ixy="0.0" ixz="0.0"
-               iyy="0.3375" iyz="0.0"
-               izz="0.4125"/>
+      <origin xyz="0 0 ${chassis_height/2}" rpy="0 0 0"/>
+      <mass value="${chassis_mass}"/>
+      <inertia
+        ixx="${chassis_mass/12.0*(chassis_width*chassis_width + chassis_height*chassis_height)}" ixy="0.0" ixz="0.0"
+        iyy="${chassis_mass/12.0*(chassis_length*chassis_length + chassis_height*chassis_height)}" iyz="0.0"
+        izz="${chassis_mass/12.0*(chassis_length*chassis_length + chassis_width*chassis_width)}"/>
     </inertial>
   </link>
-  <!-- Wheel Macro -->
-  <xacro:macro name="wheel" params="prefix suffix pos_x pos_y">
-    <link name="${prefix}_${suffix}_wheel">
+  <!-- ============================ Drive wheels ============================ -->
+  <xacro:macro name="drive_wheel" params="side reflect">
+    <link name="${side}_wheel">
       <visual>
         <origin xyz="0 0 0" rpy="${pi/2} 0 0"/>
-        <geometry>
-          <cylinder radius="${wheel_radius}" length="${wheel_width}"/>
-        </geometry>
-        <material name="black">
-          <color rgba="0.0 0.0 0.0 1.0"/>
-        </material>
+        <geometry><cylinder radius="${wheel_radius}" length="${wheel_width}"/></geometry>
+        <material name="black"><color rgba="0.05 0.05 0.05 1.0"/></material>
       </visual>
       <collision>
         <origin xyz="0 0 0" rpy="${pi/2} 0 0"/>
-        <geometry>
-          <cylinder radius="${wheel_radius}" length="${wheel_width}"/>
-        </geometry>
+        <geometry><cylinder radius="${wheel_radius}" length="${wheel_width}"/></geometry>
       </collision>
       <inertial>
-        <mass value="0.5"/>
         <origin xyz="0 0 0" rpy="${pi/2} 0 0"/>
-        <inertia ixx="0.000833" ixy="0.0" ixz="0.0"
-                 iyy="0.000833" iyz="0.0"
-                 izz="0.00125"/>
+        <mass value="${wheel_mass}"/>
+        <inertia
+          ixx="${wheel_mass/12.0*(3*wheel_radius*wheel_radius + wheel_width*wheel_width)}" ixy="0.0" ixz="0.0"
+          iyy="${wheel_mass/12.0*(3*wheel_radius*wheel_radius + wheel_width*wheel_width)}" iyz="0.0"
+          izz="${wheel_mass/2.0*wheel_radius*wheel_radius}"/>
       </inertial>
     </link>
-    <joint name="${prefix}_${suffix}_wheel_joint" type="continuous">
+    <joint name="${side}_wheel_joint" type="continuous">
       <parent link="base_link"/>
-      <child link="${prefix}_${suffix}_wheel"/>
-      <origin xyz="${pos_x} ${pos_y} ${wheel_offset_z}" rpy="0 0 0"/>
+      <child link="${side}_wheel"/>
+      <origin xyz="0 ${reflect*wheel_offset_y} 0" rpy="0 0 0"/>
       <axis xyz="0 1 0"/>
     </joint>
   </xacro:macro>
-  <!-- Instantiate the four wheels -->
-  <xacro:wheel prefix="front" suffix="left" pos_x="${wheel_offset_x}" pos_y="${wheel_offset_y}"/>
-  <xacro:wheel prefix="front" suffix="right" pos_x="${wheel_offset_x}" pos_y="${-wheel_offset_y}"/>
-  <xacro:wheel prefix="rear" suffix="left" pos_x="${-wheel_offset_x}" pos_y="${wheel_offset_y}"/>
-  <xacro:wheel prefix="rear" suffix="right" pos_x="${-wheel_offset_x}" pos_y="${-wheel_offset_y}"/>
-  <!-- IMU Sensor Link -->
+  <xacro:drive_wheel side="left"  reflect="1"/>
+  <xacro:drive_wheel side="right" reflect="-1"/>
+  <!-- ============================ Ball casters (frictionless) ============================ -->
+  <xacro:macro name="caster" params="pos reflect">
+    <link name="${pos}_caster">
+      <visual>
+        <origin xyz="0 0 0" rpy="0 0 0"/>
+        <geometry><sphere radius="${caster_radius}"/></geometry>
+        <material name="grey"><color rgba="0.4 0.4 0.4 1.0"/></material>
+      </visual>
+      <collision>
+        <origin xyz="0 0 0" rpy="0 0 0"/>
+        <geometry><sphere radius="${caster_radius}"/></geometry>
+      </collision>
+      <inertial>
+        <mass value="${caster_mass}"/>
+        <inertia ixx="${0.4*caster_mass*caster_radius*caster_radius}" ixy="0.0" ixz="0.0"
+                 iyy="${0.4*caster_mass*caster_radius*caster_radius}" iyz="0.0"
+                 izz="${0.4*caster_mass*caster_radius*caster_radius}"/>
+      </inertial>
+    </link>
+    <joint name="${pos}_caster_joint" type="fixed">
+      <parent link="base_link"/>
+      <child link="${pos}_caster"/>
+      <origin xyz="${reflect*caster_offset_x} 0 ${-(wheel_radius - caster_radius)}" rpy="0 0 0"/>
+    </joint>
+  </xacro:macro>
+  <xacro:caster pos="front" reflect="1"/>
+  <xacro:caster pos="rear"  reflect="-1"/>
+  <!-- ============================ Sensor links ============================ -->
+  <!-- IMU -->
   <link name="imu_link">
     <inertial>
       <mass value="0.01"/>
       <origin xyz="0 0 0" rpy="0 0 0"/>
-      <inertia ixx="0.00001" ixy="0.0" ixz="0.0"
-               iyy="0.00001" iyz="0.0"
-               izz="0.00001"/>
+      <inertia ixx="0.00001" ixy="0.0" ixz="0.0" iyy="0.00001" iyz="0.0" izz="0.00001"/>
     </inertial>
   </link>
@@ -93,29 +118,21 @@
     <parent link="base_link"/>
     <child link="imu_link"/>
-    <origin xyz="0 0 0" rpy="0 0 0"/>
-  </joint>
-  <!-- LiDAR Sensor Link -->
+    <origin xyz="0 0 ${chassis_height/2}" rpy="0 0 0"/>
+  </joint>
+  <!-- 3D LiDAR (roof-mounted) -->
   <link name="lidar_link">
     <visual>
       <origin xyz="0 0 0" rpy="0 0 0"/>
-      <geometry>
-        <cylinder radius="0.05" length="0.05"/>
-      </geometry>
-      <material name="red">
-        <color rgba="1.0 0.0 0.0 1.0"/>
-      </material>
+      <geometry><cylinder radius="0.05" length="0.05"/></geometry>
+      <material name="red"><color rgba="1.0 0.0 0.0 1.0"/></material>
     </visual>
     <collision>
       <origin xyz="0 0 0" rpy="0 0 0"/>
-      <geometry>
-        <cylinder radius="0.05" length="0.05"/>
-      </geometry>
+      <geometry><cylinder radius="0.05" length="0.05"/></geometry>
     </collision>
     <inertial>
       <mass value="0.1"/>
       <origin xyz="0 0 0" rpy="0 0 0"/>
-      <inertia ixx="0.0001" ixy="0.0" ixz="0.0"
-               iyy="0.0001" iyz="0.0"
-               izz="0.0001"/>
+      <inertia ixx="0.0001" ixy="0.0" ixz="0.0" iyy="0.0001" iyz="0.0" izz="0.0001"/>
     </inertial>
   </link>
@@ -123,29 +140,21 @@
     <parent link="base_link"/>
     <child link="lidar_link"/>
-    <origin xyz="0 0 ${chassis_height/2 + 0.025}" rpy="0 0 0"/>
-  </joint>
-  <!-- Camera Link -->
+    <origin xyz="0 0 ${chassis_height + 0.025}" rpy="0 0 0"/>
+  </joint>
+  <!-- RGB camera (front-facing) -->
   <link name="camera_link">
     <visual>
       <origin xyz="0 0 0" rpy="0 0 0"/>
-      <geometry>
-        <box size="0.03 0.08 0.03"/>
-      </geometry>
-      <material name="green">
-        <color rgba="0.0 1.0 0.0 1.0"/>
-      </material>
+      <geometry><box size="0.03 0.08 0.03"/></geometry>
+      <material name="green"><color rgba="0.0 1.0 0.0 1.0"/></material>
     </visual>
     <collision>
       <origin xyz="0 0 0" rpy="0 0 0"/>
-      <geometry>
-        <box size="0.03 0.08 0.03"/>
-      </geometry>
+      <geometry><box size="0.03 0.08 0.03"/></geometry>
     </collision>
     <inertial>
       <mass value="0.05"/>
       <origin xyz="0 0 0" rpy="0 0 0"/>
-      <inertia ixx="0.00001" ixy="0.0" ixz="0.0"
-               iyy="0.00001" iyz="0.0"
-               izz="0.00001"/>
+      <inertia ixx="0.00001" ixy="0.0" ixz="0.0" iyy="0.00001" iyz="0.0" izz="0.00001"/>
     </inertial>
   </link>
@@ -153,7 +162,7 @@
     <parent link="base_link"/>
     <child link="camera_link"/>
-    <origin xyz="${chassis_length/2} 0 0.02" rpy="0 0 0"/>
-  </joint>
-  <!-- Camera Optical Frame (required for ROS camera convention) -->
+    <origin xyz="${chassis_length/2} 0 ${chassis_height/2}" rpy="0 0 0"/>
+  </joint>
+  <!-- Camera optical frame (REP-103 optical convention: z forward, x right, y down) -->
   <link name="camera_optical_link"/>
   <joint name="camera_optical_joint" type="fixed">
@@ -162,95 +171,125 @@
     <origin xyz="0 0 0" rpy="${-pi/2} 0 ${-pi/2}"/>
   </joint>
-  <!-- ===================== GAZEBO PLUGINS ===================== -->
-  <!-- Gazebo properties for colors -->
+  <!-- ===================== GAZEBO (HARMONIC) MATERIALS & FRICTION ===================== -->
   <gazebo reference="base_link">
-    <material>Gazebo/Blue</material>
-  </gazebo>
-  <gazebo reference="front_left_wheel">
-    <material>Gazebo/Black</material>
+    <material>
+      <ambient>0.0 0.0 1.0 1.0</ambient>
+      <diffuse>0.0 0.0 1.0 1.0</diffuse>
+      <specular>0.1 0.1 0.1 1.0</specular>
+    </material>
+  </gazebo>
+  <gazebo reference="left_wheel">
+    <material><ambient>0.05 0.05 0.05 1.0</ambient><diffuse>0.05 0.05 0.05 1.0</diffuse></material>
     <mu1>1.0</mu1>
     <mu2>1.0</mu2>
   </gazebo>
-  <gazebo reference="front_right_wheel">
-    <material>Gazebo/Black</material>
+  <gazebo reference="right_wheel">
+    <material><ambient>0.05 0.05 0.05 1.0</ambient><diffuse>0.05 0.05 0.05 1.0</diffuse></material>
     <mu1>1.0</mu1>
     <mu2>1.0</mu2>
   </gazebo>
-  <gazebo reference="rear_left_wheel">
-    <material>Gazebo/Black</material>
-    <mu1>1.0</mu1>
-    <mu2>1.0</mu2>
-  </gazebo>
-  <gazebo reference="rear_right_wheel">
-    <material>Gazebo/Black</material>
-    <mu1>1.0</mu1>
-    <mu2>1.0</mu2>
+  <!-- Frictionless casters: they support the chassis without dragging/slipping the odometry -->
+  <gazebo reference="front_caster">
+    <material><ambient>0.4 0.4 0.4 1.0</ambient><diffuse>0.4 0.4 0.4 1.0</diffuse></material>
+    <mu1>0.0</mu1>
+    <mu2>0.0</mu2>
+  </gazebo>
+  <gazebo reference="rear_caster">
+    <material><ambient>0.4 0.4 0.4 1.0</ambient><diffuse>0.4 0.4 0.4 1.0</diffuse></material>
+    <mu1>0.0</mu1>
+    <mu2>0.0</mu2>
   </gazebo>
   <gazebo reference="lidar_link">
-    <material>Gazebo/Red</material>
+    <material><ambient>1.0 0.0 0.0 1.0</ambient><diffuse>1.0 0.0 0.0 1.0</diffuse></material>
   </gazebo>
   <gazebo reference="camera_link">
-    <material>Gazebo/Green</material>
-  </gazebo>
-  <!-- Differential Drive Plugin (4-Wheel Skid Steer) -->
+    <material><ambient>0.0 1.0 0.0 1.0</ambient><diffuse>0.0 1.0 0.0 1.0</diffuse></material>
+  </gazebo>
+  <!-- ===================== GAZEBO (HARMONIC) SYSTEM PLUGINS ===================== -->
   <gazebo>
-    <plugin name="diff_drive_controller" filename="libgazebo_ros_diff_drive.so">
-      <!-- Update rate in Hz -->
-      <update_rate>50</update_rate>
-      <!-- Wheel joints -->
-      <left_joint>front_left_wheel_joint</left_joint>
-      <left_joint>rear_left_wheel_joint</left_joint>
-      <right_joint>front_right_wheel_joint</right_joint>
-      <right_joint>rear_right_wheel_joint</right_joint>
-      <!-- Wheel separation and diameter -->
+    <!-- Differential drive: exactly two driven wheels + wheel odometry -->
+    <plugin filename="gz-sim-diff-drive-system" name="gz::sim::systems::DiffDrive">
+      <left_joint>left_wheel_joint</left_joint>
+      <right_joint>right_wheel_joint</right_joint>
       <wheel_separation>${2*wheel_offset_y}</wheel_separation>
-      <wheel_diameter>${2*wheel_radius}</wheel_diameter>
-      <!-- Limits -->
-      <max_wheel_torque>20</max_wheel_torque>
-      <max_wheel_acceleration>1.0</max_wheel_acceleration>
-      <!-- Output -->
-      <publish_odom>true</publish_odom>
-      <publish_odom_tf>true</publish_odom_tf>
-      <publish_wheel_tf>true</publish_wheel_tf>
-      <odometry_frame>odom</odometry_frame>
-      <robot_base_frame>base_footprint</robot_base_frame>
-      <!-- Topic names -->
-      <command_topic>cmd_vel</command_topic>
-      <odometry_topic>odom</odometry_topic>
+      <wheel_radius>${wheel_radius}</wheel_radius>
+      <odom_publish_frequency>50</odom_publish_frequency>
+      <max_linear_acceleration>1.0</max_linear_acceleration>
+      <min_linear_acceleration>-1.0</min_linear_acceleration>
+      <max_angular_acceleration>2.0</max_angular_acceleration>
+      <min_angular_acceleration>-2.0</min_angular_acceleration>
+      <max_linear_velocity>0.6</max_linear_velocity>
+      <min_linear_velocity>-0.6</min_linear_velocity>
+      <max_angular_velocity>1.2</max_angular_velocity>
+      <min_angular_velocity>-1.2</min_angular_velocity>
+      <topic>cmd_vel</topic>
+      <odom_topic>odom</odom_topic>
+      <tf_topic>/tf</tf_topic>
+      <frame_id>odom</frame_id>
+      <child_frame_id>base_footprint</child_frame_id>
     </plugin>
-  </gazebo>
-  <!-- IMU Sensor Plugin -->
+    <!-- Joint states for the two wheels -->
+    <plugin filename="gz-sim-joint-state-publisher-system" name="gz::sim::systems::JointStatePublisher">
+      <topic>joint_states</topic>
+      <joint_name>left_wheel_joint</joint_name>
+      <joint_name>right_wheel_joint</joint_name>
+    </plugin>
+    <!-- IMU system (drives the imu sensor below) -->
+    <plugin filename="gz-sim-imu-system" name="gz::sim::systems::Imu"/>
+    <!-- Perfect ground-truth odometry (topic only, NOT on /tf, to avoid TF conflicts) -->
+    <plugin filename="gz-sim-odometry-publisher-system" name="gz::sim::systems::OdometryPublisher">
+      <odom_frame>odom</odom_frame>
+      <robot_base_frame>base_link</robot_base_frame>
+      <odom_topic>/ground_truth</odom_topic>
+      <dimensions>3</dimensions>
+      <odom_publish_frequency>30</odom_publish_frequency>
+    </plugin>
+  </gazebo>
+  <!-- ===================== GAZEBO (HARMONIC) SENSORS ===================== -->
+  <!-- IMU sensor @ 100 Hz -->
   <gazebo reference="imu_link">
     <sensor name="imu_sensor" type="imu">
       <always_on>true</always_on>
       <update_rate>100</update_rate>
-      <plugin name="imu_plugin" filename="libgazebo_ros_imu_sensor.so">
-        <ros>
-          <namespace>/</namespace>
-          <remapping>~/out:=imu/data</remapping>
-        </ros>
-        <initial_orientation_as_reference>false</initial_orientation_as_reference>
-      </plugin>
+      <visualize>true</visualize>
+      <topic>imu/data</topic>
+      <gz_frame_id>imu_link</gz_frame_id>
+      <enable_metrics>false</enable_metrics>
+      <imu>
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